File: hardware/pcb/PCB_Sumo.kicad_sch (KiCad schematic)
At the start: 27 parts

Commit message: PCB v2 (WIP): divisor de batería en GP6, ESP32 a 15.24 mm
Parts:
- added R11: 20k, Resistor_THT:R_Axial_DIN0207_L6.3mm_D2.5mm_P10.16mm_Horizontal, symbol Device:R
- added R12: 10k, Resistor_THT:R_Axial_DIN0207_L6.3mm_D2.5mm_P10.16mm_Horizontal, symbol Device:R
Connections:
- net +7.4V: now also R11.2
- net GND: now also R12.1
- net V_BAT_SENSE: now reaches ESP32_IZQ1.9 (Pin_9)
- net V_BAT_SENSE: now also R11.1, R12.2
- no-connect marks 4 -> 3
